File: pcb/Si468x.kicad_pcb (KiCad board)
At the start: 4 copper layers, 22 x 30 mm, 60 parts, among them J1 Bus_M.2_Socket_E, J2 ANT0, Q1 BSS138, U1 TPS7A2118-DRB, U2 PCA9306, U3 74LVC1G17, U4 Si4689-A10, U5 ZD25WQ32C, Y1 19.2MHZ

Commit message: bought like that
Parts:
- renumbered FlashWP to JP1
Routing:
- net GND: vias 135 -> 134
Changed lines of the file:
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@@
 			(plot_on_all_layers_selection 0x00000000_00000000_00000000_00000000)
 			(disableapertmacros no)
-			(usegerberextensions no)
+			(usegerberextensions yes)
 			(usegerberattributes yes)
 			(usegerberadvancedattributes yes)
-			(creategerberjobfile yes)
+			(creategerberjobfile no)
 			(dashed_line_dash_ratio 12.000000)
 			(dashed_line_gap_ratio 3.000000)
@@
 			(plotpadnumbers no)
 			(hidednponfab no)
-			(sketchdnponfab no)
-			(crossoutdnponfab no)
+			(sketchdnponfab yes)
+			(crossoutdnponfab yes)
 			(subtractmaskfromsilk no)
 			(outputformat 1)
@@
 		(tags "inductor")
 		(property "Reference" "L4"
-			(at 0.615 0.7 0)
+			(at 0.613917 0.776635 0)
 			(layer "F.SilkS")
 			(effects
@@
 		(sheetname "/")
 		(sheetfile "Si468x.kicad_sch")
-		(attr smd)
+		(attr smd dnp)
 		(fp_line
 			(start -0.153641 -0.38)
@@
 		(sheetname "/")
 		(sheetfile "Si468x.kicad_sch")
-		(attr smd)
+		(attr smd dnp)
 		(fp_line
 			(start -0.153641 0.38)
@@
 		(tags "capacitor")
 		(property "Reference" "C12"
-			(at -1.3 -0.1 90)
+			(at -1.320415 -0.00462 90)
 			(layer "F.SilkS")
 			(effects
@@
 		(sheetname "/")
 		(sheetfile "Si468x.kicad_sch")
-		(attr smd)
+		(attr smd dnp)
 		(fp_line
 			(start -0.153641 0.38)
@@
 				(font
 					(size 0.5 0.5)
-					(thickness 0.5)
+					(thickness 0.125)
 				)
 			)
@@
 		(fp_poly
 			(pts
-				(xy -2.14 -0.98) (xy -2.47 -0.74) (xy -2.47 -1.22)
+				(xy -1.49 -1.94) (xy -1.73 -2.27) (xy -1.25 -2.27)
 			)
 			(stroke
@@
 		(descr "SMD Solder Jumper, 1x1.5mm, rounded Pads, 0.3mm gap, open")
 		(tags "solder jumper open")
-		(property "Reference" "FlashWP"
+		(property "Reference" "JP1"
 			(at 0 1.8 0)
 			(layer "B.SilkS")
@@
 		)
 	)
-	(gr_rect
-		(start 138 82.6)
-		(end 159.1 99.1)
-		(stroke
-			(width 0.1)
-			(type solid)
-		)
-		(fill no)
-		(layer "Dwgs.User")
-	)
 	(segment
 		(start 145.9 104.4)
@@
 	)
 	(via
-		(at 138.5 81)
+		(at 138.3 81)
 		(size 0.6)
 		(drill 0.3)
@@
 	)
 	(via
-		(at 139.34105 88.139862)
-		(size 0.6)
-		(drill 0.3)
-		(layers "F.Cu" "B.Cu")
-		(free yes)
-		(net 2)
-	)
-	(via
 		(at 149 99.75)
 		(size 0.6)
@@
 			)
 		)
+	)
+	(zone
+		(net 0)
+		(net_name "")
+		(layer "B.Cu")
+		(hatch edge 0.5)
+		(connect_pads
+			(clearance 0)
+		)
+		(min_thickness 0.25)
+		(filled_areas_thickness no)
+		(keepout
+			(tracks allowed)
+			(vias allowed)
+			(pads allowed)
+			(copperpour not_allowed)
+			(footprints allowed)
+		)
+		(placement
+			(enabled no)
+			(sheetname "/")
+		)
+		(fill
+			(thermal_gap 0.5)
+			(thermal_bridge_width 0.5)
+		)
+		(polygon
+			(pts
+				(xy 151 97.25) (xy 151 94.25) (xy 153.25 92.25) (xy 154.5 93.5) (xy 154.5 95) (xy 152.25 97.25)
+			)
+		)
