File: pcb/Si468x.kicad_sch (KiCad schematic)
At the start: 0 parts

Commit message: main PCB basicly finished
Parts:
- added C1: 1u, Capacitor_SMD:C_0603_1608Metric, symbol Device:C
- added C2, C3: 4.7u, Capacitor_SMD:C_0603_1608Metric, symbol Device:C
- added C4: 100p, Capacitor_SMD:C_0402_1005Metric, symbol Device:C
- added C5: 0.1uF, Capacitor_SMD:C_0402_1005Metric, symbol Device:C
- added J1: Bus_M.2_Socket_E, Connector_PCBEdge:M.2_2230-xx-E, symbol Connector:Bus_M.2_Socket_E
- added J5: RFShield_TwoPieces, symbol Device:RFShield_TwoPieces
- added L1: BLM18PG, Inductor_SMD:L_0603_1608Metric, symbol Device:L
- added Q1: BSS138, Package_TO_SOT_SMD:SOT-23, symbol Transistor_FET:BSS138
- added R1, R2, R3: 33R, Resistor_SMD:R_0402_1005Metric, symbol Device:R
- added R10, R11, R5, R8: 2.2k, Resistor_SMD:R_0402_1005Metric, symbol Device:R
- added R4, R7: 10k, Resistor_SMD:R_0402_1005Metric, symbol Device:R
- added R6: 100k, Resistor_SMD:R_0402_1005Metric, symbol Device:R
- added R9: 200k, Resistor_SMD:R_0402_1005Metric, symbol Device:R
- added TP1: 3V3, TestPoint:TestPoint_Pad_D1.0mm, symbol Connector:TestPoint
- added TP2: 1V8, TestPoint:TestPoint_Pad_D1.0mm, symbol Connector:TestPoint
- added TP5: GND, TestPoint:TestPoint_Pad_D1.0mm, symbol Connector:TestPoint
- added U1: TPS7A2118-DRB, library:Texas_DRB_VSON_8, symbol Si468x:TPS7A21-Q1-DRB
- added U2: PCA9306, Package_SO:VSSOP-8_2.3x2mm_P0.5mm, symbol Interface:PCA9306
- added U3: 74LVC1G17, Package_TO_SOT_SMD:Texas_R-PDSO-G5_DCK-5, symbol 74xGxx:74LVC1G17
Connections:
- new net: J1.60 (I2C_CLK), R5.2, U2.6 (SCL2)
- new net: C4.1, R9.2, U2.7 (VREF2), U2.8 (EN)
- new net: J1.58 (I2C_DATA), R8.2, U2.5 (SDA2)
- new net: J1.12 (PCM_IN/I2S_SD_IN), R3.1
- new net: J1.10 (PCM_SYNC/I2S_WS), R2.1
- new net: J1.62 (~{ALERT}), Q1.3 (D), R4.1
- new net: J1.8 (PCM_CLK/I2S_SCK), R1.1
- new net: C1.1, L1.2, U1.5 (EN), U1.8 (IN)
- new net +1V8: C2.1, C5.2, R10.1, R11.1, R7.1, TP2.1, U1.1 (OUT), U2.2 (VREF1), U3.5 (VCC)
- new net +3V3: C3.2, J1.2 (3.3V), J1.4 (3.3V), J1.72 (3.3V), J1.74 (3.3V), L1.1, R4.2, R5.1, R6.2, R8.1, R9.1, TP1.1
- new net GND: C1.2, C2.2, C3.1, C4.2, C5.1, J1.1 (GND), J1.18 (GND), J1.33 (GND), J1.39 (GND), J1.45 (GND), J1.51 (GND), J1.57 (GND), J1.63 (GND), J1.69 (GND), J1.7 (GND), J1.75 (GND), J5.1 (Shield), TP5.1, U1.2 (NC), U1.3 (NC), U1.4 (GND), U1.6 (NC), U1.7 (NC), U1.9 (EP), U2.1 (GND), U3.3 (GND)
- new net Si4689/DCLK: R1.2
- new net Si4689/DFS: R2.2
- new net Si4689/DOUT: R3.2
- new net Si4689/INTB: Q1.1 (G), Q1.2 (S), R7.2
- new net Si4689/SCL: R11.2, U2.3 (SCL1)
- new net Si4689/SDA: R10.2, U2.4 (SDA1)
- new net Si4689/~{RST}: U3.4
- new net ~{W_DISABLE1}: J1.56 (~{W_DISABLE1}), R6.1, U3.2
- no-connect marks 0 -> 42
Other:
- added sheet Si4689 (Si4689.kicad_sch)

Commit message: bought like that
Parts:
- removed J5: RFShield_TwoPieces, symbol Device:RFShield_TwoPieces
- R4, R5, R8: now not fitted
Other:
- moved on the sheet: TP5
Changed lines of the file:
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@@
 	(wire
 		(pts
+			(xy 71.12 182.88) (xy 67.31 182.88)
+		)
+		(stroke
+			(width 0)
+			(type default)
+		)
+	)
+	(wire
+		(pts
 			(xy 256.54 44.45) (xy 243.84 44.45)
 		)
@@
 		(in_bom yes)
 		(on_board yes)
-		(dnp no)
+		(dnp yes)
 		(fields_autoplaced yes)
 		(property "Reference" "R5"
@@
 		(in_bom yes)
 		(on_board yes)
-		(dnp no)
+		(dnp yes)
 		(fields_autoplaced yes)
 		(property "Reference" "R8"
@@
 	(symbol
 		(lib_id "power:GND")
-		(at 48.26 85.09 0)
-		(unit 1)
-		(exclude_from_sim no)
-		(in_bom yes)
-		(on_board yes)
-		(dnp no)
-		(fields_autoplaced yes)
-		(property "Reference" "#PWR037"
-			(at 48.26 91.44 0)
-			(effects
-				(font
-					(size 1.27 1.27)
-				)
-				(hide yes)
-			)
-		)
-		(property "Value" "GND"
-			(at 48.26 90.17 0)
-			(effects
-				(font
-					(size 1.27 1.27)
-				)
-			)
-		)
-		(property "Footprint" ""
-			(at 48.26 85.09 0)
-			(effects
-				(font
-					(size 1.27 1.27)
-				)
-				(hide yes)
-			)
-		)
-		(property "Datasheet" ""
-			(at 48.26 85.09 0)
-			(effects
-				(font
-					(size 1.27 1.27)
-				)
-				(hide yes)
-			)
-		)
-		(property "Description" "Power symbol creates a global label with name \"GND\" , ground"
-			(at 48.26 85.09 0)
-			(effects
-				(font
-					(size 1.27 1.27)
-				)
-				(hide yes)
-			)
-		)
-		(pin "1"
-		)
-		(instances
-			(project "Si468x"
-				(path "/cee16205-ad08-4662-b2ce-24dda8a7e2eb"
-					(reference "#PWR037")
-					(unit 1)
-				)
-			)
-		)
-	)
-	(symbol
-		(lib_id "power:GND")
 		(at 241.3 71.12 0)
 		(unit 1)
@@
 		(in_bom yes)
 		(on_board yes)
-		(dnp no)
+		(dnp yes)
 		(fields_autoplaced yes)
 		(property "Reference" "R4"
@@
 	)
 	(symbol
+		(lib_id "power:PWR_FLAG")
+		(at 67.31 182.88 180)
+		(unit 1)
+		(exclude_from_sim no)
+		(in_bom yes)
+		(on_board yes)
+		(dnp no)
+		(fields_autoplaced yes)
+		(property "Reference" "#FLG01"
+			(at 67.31 184.785 0)
+			(effects
+				(font
+					(size 1.27 1.27)
+				)
+				(hide yes)
+			)
+		)
+		(property "Value" "PWR_FLAG"
+			(at 67.31 187.96 0)
+			(effects
+				(font
+					(size 1.27 1.27)
+				)
+			)
+		)
+		(property "Footprint" ""
+			(at 67.31 182.88 0)
+			(effects
+				(font
+					(size 1.27 1.27)
+				)
+				(hide yes)
+			)
+		)
+		(property "Datasheet" "~"
+			(at 67.31 182.88 0)
+			(effects
+				(font
+					(size 1.27 1.27)
+				)
+				(hide yes)
+			)
+		)
+		(property "Description" "Special symbol for telling ERC where power comes from"
+			(at 67.31 182.88 0)
+			(effects
+				(font
+					(size 1.27 1.27)
+				)
+				(hide yes)
+			)
+		)
+		(pin "1"
+		)
+		(instances
+			(project "Si468x"
+				(path "/cee16205-ad08-4662-b2ce-24dda8a7e2eb"
+					(reference "#FLG01")
+					(unit 1)
+				)
+			)
+		)
+	)
+	(symbol
 		(lib_id "Connector:TestPoint")
 		(at 67.31 163.83 0)
@@
 	(symbol
 		(lib_id "Connector:TestPoint")
-		(at 67.31 182.88 180)
+		(at 71.12 182.88 270)
 		(unit 1)
 		(exclude_from_sim no)
@@
 		(fields_autoplaced yes)
 		(property "Reference" "TP5"
-			(at 69.85 184.9119 0)
+			(at 76.2 181.6099 90)
 			(effects
 				(font
 					(size 1.27 1.27)
 				)
-				(justify right)
+				(justify left)
 			)
 		)
 		(property "Value" "GND"
-			(at 69.85 187.4519 0)
+			(at 76.2 184.1499 90)
 			(effects
 				(font
 					(size 1.27 1.27)
 				)
-				(justify right)
+				(justify left)
 			)
 		)
 		(property "Footprint" "TestPoint:TestPoint_Pad_D1.0mm"
-			(at 62.23 182.88 0)
+			(at 71.12 187.96 0)
 			(effects
 				(font
@@
 		)
 		(property "Datasheet" "~"
-			(at 62.23 182.88 0)
+			(at 71.12 187.96 0)
 			(effects
 				(font
@@
 		)
 		(property "Description" "test point"
-			(at 67.31 182.88 0)
+			(at 71.12 182.88 0)
 			(effects
 				(font
@@
 					(unit 1)
 				)
-			)
-		)
-	)
-	(symbol
-		(lib_id "Device:RFShield_TwoPieces")
-		(at 48.26 74.93 0)
-		(unit 1)
-		(exclude_from_sim no)
-		(in_bom yes)
-		(on_board yes)
-		(dnp no)
-		(fields_autoplaced yes)
-		(property "Reference" "J5"
-			(at 67.31 71.7549 0)
-			(effects
-				(font
-					(size 1.27 1.27)
-				)
-				(justify left)
-			)
-		)
-		(property "Value" "RFShield_TwoPieces"
-			(at 67.31 74.2949 0)
-			(effects
-				(font
-					(size 1.27 1.27)
-				)
-				(justify left)
-			)
-		)
-		(property "Footprint" ""
-			(at 48.26 77.47 0)
-			(effects
-				(font
-					(size 1.27 1.27)
-				)
-				(hide yes)
-			)
-		)
-		(property "Datasheet" "~"
-			(at 48.26 77.47 0)
-			(effects
-				(font
-					(size 1.27 1.27)
-				)
-				(hide yes)
-			)
-		)
-		(property "Description" "Two-piece EMI RF shielding cabinet"
-			(at 48.26 74.93 0)
-			(effects
-				(font
-					(size 1.27 1.27)
-				)
-				(hide yes)
-			)
-		)
-		(pin "1"
-		)
-		(instances
-			(project "Si468x"
-				(path "/cee16205-ad08-4662-b2ce-24dda8a7e2eb"
-					(reference "J5")
-					(unit 1)
-				)
